File: hw/io.kicad_sch (KiCad schematic)
At the start: 12 parts, among them J1 Conn_02x08_Odd_Even, J3 Conn_02x08_Odd_Even, U11 74HC138, U5 74HC86, U6 74HC245, U7 74HC245, U8 74HC02, U9 74HC00

Commit message: Work on scmenatic and PCB
Parts:
- removed J1, J3: Conn_02x08_Odd_Even, Connector_PinHeader_2.54mm:PinHeader_2x08_P2.54mm_Vertical, symbol Connector_Generic:Conn_02x08_Odd_Even
- removed U7 (x2): 74HC245, Package_DIP:DIP-20_W7.62mm_Socket_LongPads, symbol 74xx:74HC245
- added C6 (x5): Dec_Cap, Capacitor_THT:C_Disc_D3.0mm_W1.6mm_P2.50mm, symbol z80mgc:Dec_Cap
- added J1, J3, J4: Conn_02x08_Counter_Clockwise, z80mgc:PinHeader_2x08_P2.54mm_Vertical, symbol Connector_Generic:Conn_02x08_Counter_Clockwise
- added U7: 74HC245, Package_DIP:DIP-20_W7.62mm_Socket_LongPads, symbol 74xx:74HC245
Connections:
- net +5V: now also C6.1, C6.1, C6.1, C6.1, C6.1, J3.15 (Pin_15), J3.16 (Pin_16), U7.20 (VCC)
- net DATA0: now also U7.2 (A0)
- net DATA1: now also U7.3 (A1)
- net DATA2: now also U7.4 (A2)
- net DATA3: now also U7.5 (A3)
- net DATA4: now also U7.6 (A4)
- net DATA5: now also U7.7 (A5)
- net DATA6: now also U7.8 (A6)
- net DATA7: now also U7.9 (A7)
- net GND: now also C6.2, C6.2, C6.2, C6.2, C6.2, J3.13 (Pin_13), J3.14 (Pin_14), U7.1 (A->B), U7.10 (GND)
- net ~{RD}: now also J3.9 (Pin_9)
- net ~{WR}: now also J3.10 (Pin_10)
- net at U6.18 (B0): now also J1.1 (Pin_1)
- net at U6.17 (B1): now also J1.2 (Pin_2)
- net at U6.16 (B2): now also J1.3 (Pin_3)
- net at U6.15 (B3): now also J1.4 (Pin_4)
- net at U6.14 (B4): now also J1.5 (Pin_5)
- net at U6.13 (B5): now also J1.6 (Pin_6)
- net at U6.12 (B6): now also J1.7 (Pin_7)
- net at U6.11 (B7): now also J1.8 (Pin_8)
- net at U6.18 (B0): now also J3.1 (Pin_1)
- net at U6.17 (B1): now also J3.2 (Pin_2)
- net at U6.16 (B2): now also J3.3 (Pin_3)
- net at U6.15 (B3): now also J3.4 (Pin_4)
- net at U6.14 (B4): now also J3.5 (Pin_5)
- net at U6.13 (B5): now also J3.6 (Pin_6)
- net at U6.12 (B6): now also J3.7 (Pin_7)
- net at U6.11 (B7): now also J3.8 (Pin_8)
- net at U11.13 (~{Y2}): now also U7.19 (CE)
- new net: J4.1 (Pin_1), U7.18 (B0)
- new net: J4.2 (Pin_2), U7.17 (B1)
- new net: J4.3 (Pin_3), U7.16 (B2)
- new net: J4.4 (Pin_4), U7.15 (B3)
- new net: J4.5 (Pin_5), U7.14 (B4)
- new net: J4.6 (Pin_6), U7.13 (B5)
- new net: J4.7 (Pin_7), U7.12 (B6)
- new net: J4.8 (Pin_8), U7.11 (B7)
- new net ~{CLK}: J3.11 (Pin_11), J3.12 (Pin_12)
- no-connect marks 1 -> 5
Other:
- moved on the sheet: U6

Commit message: Work on scmenatic and PCB
Parts:
- removed C6: Dec_Cap, Capacitor_THT:C_Disc_D3.0mm_W1.6mm_P2.50mm, symbol z80mgc:Dec_Cap
- removed J3: Conn_02x08_Counter_Clockwise, z80mgc:PinHeader_2x08_P2.54mm_Vertical, symbol Connector_Generic:Conn_02x08_Counter_Clockwise
- removed U5: 74HC86, Package_DIP:DIP-14_W7.62mm_Socket_LongPads, symbol 74xx:74HC86
- removed U6: 74HC245, Package_DIP:DIP-20_W7.62mm_Socket_LongPads, symbol 74xx:74HC245
- removed U8: 74HC02, Package_DIP:DIP-14_W7.62mm_Socket_LongPads, symbol 74xx:74HC02
- removed U9: 74HC00, Package_DIP:DIP-14_W7.62mm_Socket_LongPads, symbol 74xx:74HC00
- added J6: IO_EXP, z80mgc:PinHeader_2x08_P2.54mm_Vertical, symbol Connector_Generic:Conn_02x08_Counter_Clockwise
- added RN1 (x2): R_Network08, Resistor_THT:R_Array_SIP9, symbol Device:R_Network08
- added U16: 74HC00, Package_DIP:DIP-14_W7.62mm_Socket_LongPads, symbol 74xx:74HC00
- added U17: 74HC02, Package_DIP:DIP-14_W7.62mm_Socket_LongPads, symbol 74xx:74HC02
- added U7: 74HC86, Package_DIP:DIP-14_W7.62mm_Socket_LongPads, symbol 74xx:74HC86
- C6: value Dec_Cap -> 0.1uF
- C6: value Dec_Cap -> F
- J1: renamed from J4; value Conn_02x08_Counter_Clockwise -> IO_A
- J3: renamed from J1; value Conn_02x08_Counter_Clockwise -> IO_BTN
Connections:
- net +5V: now also J6.11 (Pin_11), RN1.1 (common), RN1.1 (common)
- net ADDR0: now also J6.10 (Pin_10)
- net ADDR1: now also U7.1
- net DATA0: now also J6.1 (Pin_1)
- net DATA1: now also J6.2 (Pin_2)
- net DATA2: now also J6.3 (Pin_3)
- net DATA3: now also J6.4 (Pin_4)
- net DATA4: now also J6.5 (Pin_5)
- net DATA5: now also J6.6 (Pin_6)
- net DATA6: now also J6.7 (Pin_7)
- net DATA7: now also J6.8 (Pin_8)
- net GND: now also J1.10 (Pin_10), J1.11 (Pin_11), J1.12 (Pin_12), J1.13 (Pin_13), J1.14 (Pin_14), J1.15 (Pin_15), J1.16 (Pin_16), J1.9 (Pin_9), J3.10 (Pin_10), J3.11 (Pin_11), J3.12 (Pin_12), J3.13 (Pin_13), J3.14 (Pin_14), J3.15 (Pin_15), J3.16 (Pin_16), J3.9 (Pin_9), J6.9 (Pin_9); no longer U7.1 (A->B)
- net ~{IORQ}: now also J6.12 (Pin_12)
- net ~{RD}: now also U7.1 (A->B), J6.14 (Pin_14), U16.9
- net ~{WR}: now also J6.13 (Pin_13), U16.10, U7.2
- net at U11.15 (~{Y0}): now also U17.9
- net at DS1.6 (E): now also U17.10
- net at J3.8 (Pin_8), U6.11 (B7): now also RN1.2 (R1)
- net at J3.7 (Pin_7), U6.12 (B6): now also RN1.3 (R2)
- net at J3.6 (Pin_6), U6.13 (B5): now also RN1.4 (R3)
- net at J3.5 (Pin_5), U6.14 (B4): now also RN1.5 (R4)
- net at J3.4 (Pin_4), U6.15 (B3): now also RN1.6 (R5)
- net at J3.3 (Pin_3), U6.16 (B2): now also RN1.7 (R6)
- net at J3.2 (Pin_2), U6.17 (B1): now also RN1.8 (R7)
- net at J3.1 (Pin_1), U6.18 (B0): now also RN1.9 (R8)
- net at J1.1 (Pin_1), U7.18 (B0): now also RN1.9 (R8)
- net at J1.2 (Pin_2), U7.17 (B1): now also RN1.8 (R7)
- net at J1.3 (Pin_3), U7.16 (B2): now also RN1.7 (R6)
- net at J1.4 (Pin_4), U7.15 (B3): now also RN1.6 (R5)
- net at J1.5 (Pin_5), U7.14 (B4): now also RN1.5 (R4)
- net at J1.6 (Pin_6), U7.13 (B5): now also RN1.4 (R3)
- net at J1.7 (Pin_7), U7.12 (B6): now also RN1.3 (R2)
- net at J1.8 (Pin_8), U7.11 (B7): now also RN1.2 (R1)
- net at U11.12 (~{Y3}): now also J6.16 (Pin_16)
- net at U11.6 (E3): now also U16.8
- net at U11.11 (~{Y4}): now also J6.15 (Pin_15)
- new net: U17.8, U7.3
- no-connect marks 5 -> 3
Other:
- moved on the sheet: C6, J1, J3, U6, U7

Commit message: Snake working with framebuffer
Parts:
- removed RN1 (x2): R_Network08, Resistor_THT:R_Array_SIP9, symbol Device:R_Network08
- added RN1 (x2): 10k, Resistor_THT:R_Array_SIP9, symbol Device:R_Network08
Connections:
- net +5V: now also RN1.1 (common), RN1.1 (common)
- net at J3.8 (Pin_8), U6.11 (B7): now also RN1.9 (R8)
- net at J3.7 (Pin_7), U6.12 (B6): now also RN1.8 (R7)
- net at J3.6 (Pin_6), U6.13 (B5): now also RN1.7 (R6)
- net at J3.5 (Pin_5), U6.14 (B4): now also RN1.6 (R5)
- net at J3.4 (Pin_4), U6.15 (B3): now also RN1.5 (R4)
- net at J3.3 (Pin_3), U6.16 (B2): now also RN1.4 (R3)
- net at J3.2 (Pin_2), U6.17 (B1): now also RN1.3 (R2)
- net at J3.1 (Pin_1), U6.18 (B0): now also RN1.2 (R1)
- net at J1.1 (Pin_1), U7.18 (B0): now also RN1.2 (R1)
- net at J1.2 (Pin_2), U7.17 (B1): now also RN1.3 (R2)
- net at J1.3 (Pin_3), U7.16 (B2): now also RN1.4 (R3)
- net at J1.4 (Pin_4), U7.15 (B3): now also RN1.5 (R4)
- net at J1.5 (Pin_5), U7.14 (B4): now also RN1.6 (R5)
- net at J1.6 (Pin_6), U7.13 (B5): now also RN1.7 (R6)
- net at J1.7 (Pin_7), U7.12 (B6): now also RN1.8 (R7)
- net at J1.8 (Pin_8), U7.11 (B7): now also RN1.9 (R8)
- net DISP_EN: now reaches DS1.6 (E), U17.10
Changed lines of the file:
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@@
   (junction (at 251.46 81.28) (diameter 0) (color 0 0 0 0)
+  )
+  (junction (at 111.76 26.67) (diameter 0) (color 0 0 0 0)
   )
   (junction (at 256.54 76.2) (diameter 0) (color 0 0 0 0)
@@
     (stroke (width 0) (type default))
   )
+  (wire (pts (xy 109.22 26.67) (xy 111.76 26.67))
+    (stroke (width 0) (type default))
+  )
   (wire (pts (xy 156.21 29.21) (xy 156.21 33.02))
     (stroke (width 0) (type default))
@@
     )
   )
+  (global_label "DISP_EN" (shape input) (at 109.22 26.67 180) (fields_autoplaced)
+    (effects (font (size 1.27 1.27)) (justify right))
+    (property "Intersheetrefs" "${INTERSHEET_REFS}" (at 98.5128 26.67 0)
+      (effects (font (size 1.27 1.27)) (justify right) hide)
+    )
+  )
   (symbol (lib_id "power:+5V") (at 95.25 130.81 0) (unit 1)
     (in_bom yes) (on_board yes) (dnp no) (fields_autoplaced)
@@
     )
   )
-  (symbol (lib_id "power:+5V") (at 238.76 63.5 0) (unit 1)
+  (symbol (lib_id "power:+5V") (at 256.54 63.5 0) (unit 1)
     (in_bom yes) (on_board yes) (dnp no)
-    (property "Reference" "#PWR037" (at 238.76 67.31 0)
-      (effects (font (size 1.27 1.27)) hide)
-    )
-    (property "Value" "+5V" (at 234.95 62.23 0)
-      (effects (font (size 1.27 1.27)))
-    )
-    (property "Footprint" "" (at 238.76 63.5 0)
-      (effects (font (size 1.27 1.27)) hide)
-    )
-    (property "Datasheet" "" (at 238.76 63.5 0)
+    (property "Reference" "#PWR037" (at 256.54 67.31 0)
+      (effects (font (size 1.27 1.27)) hide)
+    )
+    (property "Value" "+5V" (at 252.73 62.23 0)
+      (effects (font (size 1.27 1.27)))
+    )
+    (property "Footprint" "" (at 256.54 63.5 0)
+      (effects (font (size 1.27 1.27)) hide)
+    )
+    (property "Datasheet" "" (at 256.54 63.5 0)
       (effects (font (size 1.27 1.27)) hide)
     )
@@
         )
         (path "/a0755aec-b457-49e5-8300-11792eab574c/15070439-6afa-45c0-9285-2a6cc055421b"
-          (reference "U2") (unit 3)
+          (reference "U2") (unit 4)
         )
       )
@@
         (path "/a0755aec-b457-49e5-8300-11792eab574c/15070439-6afa-45c0-9285-2a6cc055421b"
           (reference "#PWR031") (unit 1)
+        )
+      )
+    )
+  )
+  (symbol (lib_id "Device:R_Network08") (at 246.38 68.58 0) (mirror y) (unit 1)
+    (in_bom yes) (on_board yes) (dnp no)
+    (property "Reference" "RN1" (at 236.22 68.199 0)
+      (effects (font (size 1.27 1.27)) (justify left))
+    )
+    (property "Value" "10k" (at 236.22 70.739 0)
+      (effects (font (size 1.27 1.27)) (justify left))
+    )
+    (property "Footprint" "Resistor_THT:R_Array_SIP9" (at 234.315 68.58 90)
+      (effects (font (size 1.27 1.27)) hide)
+    )
+    (property "Datasheet" "http://www.vishay.com/docs/31509/csc.pdf" (at 246.38 68.58 0)
+      (effects (font (size 1.27 1.27)) hide)
+    )
+    (pin "1")
+    (pin "2")
+    (pin "3")
+    (pin "4")
+    (pin "5")
+    (pin "6")
+    (pin "7")
+    (pin "8")
+    (pin "9")
+    (instances
+      (project "z80mgc"
+        (path "/a0755aec-b457-49e5-8300-11792eab574c/0d4dd755-7db3-45ba-b967-0ba9d5a2f689"
+          (reference "RN1") (unit 1)
+        )
+        (path "/a0755aec-b457-49e5-8300-11792eab574c/15070439-6afa-45c0-9285-2a6cc055421b"
+          (reference "RN2") (unit 1)
         )
       )
@@
     )
   )
-  (symbol (lib_id "power:+5V") (at 238.76 16.51 0) (unit 1)
+  (symbol (lib_id "power:+5V") (at 256.54 16.51 0) (unit 1)
     (in_bom yes) (on_board yes) (dnp no)
-    (property "Reference" "#PWR044" (at 238.76 20.32 0)
-      (effects (font (size 1.27 1.27)) hide)
-    )
-    (property "Value" "+5V" (at 234.95 15.24 0)
-      (effects (font (size 1.27 1.27)))
-    )
-    (property "Footprint" "" (at 238.76 16.51 0)
-      (effects (font (size 1.27 1.27)) hide)
-    )
-    (property "Datasheet" "" (at 238.76 16.51 0)
+    (property "Reference" "#PWR044" (at 256.54 20.32 0)
+      (effects (font (size 1.27 1.27)) hide)
+    )
+    (property "Value" "+5V" (at 252.73 15.24 0)
+      (effects (font (size 1.27 1.27)))
+    )
+    (property "Footprint" "" (at 256.54 16.51 0)
+      (effects (font (size 1.27 1.27)) hide)
+    )
+    (property "Datasheet" "" (at 256.54 16.51 0)
       (effects (font (size 1.27 1.27)) hide)
     )
@@
         (path "/a0755aec-b457-49e5-8300-11792eab574c/15070439-6afa-45c0-9285-2a6cc055421b"
           (reference "#PWR044") (unit 1)
-        )
-      )
-    )
-  )
-  (symbol (lib_id "Device:R_Network08") (at 248.92 21.59 0) (unit 1)
-    (in_bom yes) (on_board yes) (dnp no) (fields_autoplaced)
-    (property "Reference" "RN1" (at 259.08 21.209 0)
-      (effects (font (size 1.27 1.27)) (justify left))
-    )
-    (property "Value" "R_Network08" (at 259.08 23.749 0)
-      (effects (font (size 1.27 1.27)) (justify left))
-    )
-    (property "Footprint" "Resistor_THT:R_Array_SIP9" (at 260.985 21.59 90)
-      (effects (font (size 1.27 1.27)) hide)
-    )
-    (property "Datasheet" "http://www.vishay.com/docs/31509/csc.pdf" (at 248.92 21.59 0)
-      (effects (font (size 1.27 1.27)) hide)
-    )
-    (pin "1")
-    (pin "2")
-    (pin "3")
-    (pin "4")
-    (pin "5")
-    (pin "6")
-    (pin "7")
-    (pin "8")
-    (pin "9")
-    (instances
-      (project "z80mgc"
-        (path "/a0755aec-b457-49e5-8300-11792eab574c/0d4dd755-7db3-45ba-b967-0ba9d5a2f689"
-          (reference "RN1") (unit 1)
-        )
-        (path "/a0755aec-b457-49e5-8300-11792eab574c/15070439-6afa-45c0-9285-2a6cc055421b"
-          (reference "RN1") (unit 1)
         )
       )
@@
     )
   )
+  (symbol (lib_id "Device:R_Network08") (at 246.38 21.59 0) (mirror y) (unit 1)
+    (in_bom yes) (on_board yes) (dnp no)
+    (property "Reference" "RN1" (at 236.22 21.209 0)
+      (effects (font (size 1.27 1.27)) (justify left))
+    )
+    (property "Value" "10k" (at 236.22 23.749 0)
+      (effects (font (size 1.27 1.27)) (justify left))
+    )
+    (property "Footprint" "Resistor_THT:R_Array_SIP9" (at 234.315 21.59 90)
+      (effects (font (size 1.27 1.27)) hide)
+    )
+    (property "Datasheet" "http://www.vishay.com/docs/31509/csc.pdf" (at 246.38 21.59 0)
+      (effects (font (size 1.27 1.27)) hide)
+    )
+    (pin "1")
+    (pin "2")
+    (pin "3")
+    (pin "4")
+    (pin "5")
+    (pin "6")
+    (pin "7")
+    (pin "8")
+    (pin "9")
+    (instances
+      (project "z80mgc"
+        (path "/a0755aec-b457-49e5-8300-11792eab574c/0d4dd755-7db3-45ba-b967-0ba9d5a2f689"
+          (reference "RN1") (unit 1)
+        )
+        (path "/a0755aec-b457-49e5-8300-11792eab574c/15070439-6afa-45c0-9285-2a6cc055421b"
+          (reference "RN1") (unit 1)
+        )
+      )
+    )
+  )
   (symbol (lib_id "power:GND") (at 275.59 49.53 0) (unit 1)
     (in_bom yes) (on_board yes) (dnp no)
@@
         )
         (path "/a0755aec-b457-49e5-8300-11792eab574c/15070439-6afa-45c0-9285-2a6cc055421b"
-          (reference "U4") (unit 3)
+          (reference "U4") (unit 4)
         )
       )
@@
         )
       )
-    )
-  )
-  (symbol (lib_id "Device:R_Network08") (at 248.92 68.58 0) (unit 1)
-    (in_bom yes) (on_board yes) (dnp no) (fields_autoplaced)
-    (property "Reference" "RN1" (at 259.08 68.199 0)
-      (effects (font (size 1.27 1.27)) (justify left))
-    )
-    (property "Value" "R_Network08" (at 259.08 70.739 0)
-      (effects (font (size 1.27 1.27)) (justify left))
-    )
-    (property "Footprint" "Resistor_THT:R_Array_SIP9" (at 260.985 68.58 90)
-      (effects (font (size 1.27 1.27)) hide)
-    )
-    (property "Datasheet" "http://www.vishay.com/docs/31509/csc.pdf" (at 248.92 68.58 0)
-      (effects (font (size 1.27 1.27)) hide)
-    )
-    (pin "1")
-    (pin "2")
-    (pin "3")
-    (pin "4")
-    (pin "5")
-    (pin "6")
-    (pin "7")
-    (pin "8")
-    (pin "9")
-    (instances
-      (project "z80mgc"
-        (path "/a0755aec-b457-49e5-8300-11792eab574c/0d4dd755-7db3-45ba-b967-0ba9d5a2f689"
-          (reference "RN1") (unit 1)
-        )
-        (path "/a0755aec-b457-49e5-8300-11792eab574c/15070439-6afa-45c0-9285-2a6cc055421b"
-          (reference "RN2") (unit 1)
-        )
-      )

Commit message: Lots of work on Kicad, and gave up on PCB
Parts:
- added RN5, RN6: 1k, Resistor_THT:R_Array_SIP7, symbol Device:R_Network06
Connections:
- net +5V: now also RN5.1 (common), RN6.1 (common)
- net GND: no longer J1.11 (Pin_11), J1.12 (Pin_12), J1.13 (Pin_13), J1.14 (Pin_14), J1.15 (Pin_15), J1.16 (Pin_16), J3.11 (Pin_11), J3.12 (Pin_12), J3.13 (Pin_13), J3.14 (Pin_14), J3.15 (Pin_15), J3.16 (Pin_16)
- new net: J3.16 (Pin_16), RN5.2 (R1)
- new net: J3.15 (Pin_15), RN5.3 (R2)
- new net: J3.14 (Pin_14), RN5.4 (R3)
- new net: J3.13 (Pin_13), RN5.5 (R4)
- new net: J3.12 (Pin_12), RN5.6 (R5)
- new net: J3.11 (Pin_11), RN5.7 (R6)
- new net: J1.11 (Pin_11), RN6.7 (R6)
- new net: J1.12 (Pin_12), RN6.6 (R5)
- new net: J1.13 (Pin_13), RN6.5 (R4)
- new net: J1.14 (Pin_14), RN6.4 (R3)
- new net: J1.15 (Pin_15), RN6.3 (R2)
- new net: J1.16 (Pin_16), RN6.2 (R1)
Other:
- moved on the sheet: C6, J1, J3, RN1, U6, U7
