File: hw/z80mgc.kicad_pcb (KiCad board)
At the start: 2 copper layers, 180 x 120 mm, 58 parts, among them J1 Conn_02x08_Odd_Even, J2 Conn_01x02, J3 Conn_02x08_Odd_Even, U1 Z80CPU, U10 74HC00, U11 74HC138, U12 74HC245, U13 74HC245, U14 NE555P, U2 28C256, U3 28C256, U4 71256, U5 74HC86, U6 74HC245, U7 74HC245, U8 74HC02, U9 74HC00, Y1 Crystal

Commit message: Work on scmenatic and PCB
Parts:
- removed U13: 74HC245, Package_DIP:DIP-20_W7.62mm_Socket_LongPads
- added C10: Dec_Cap, Capacitor_THT:C_Disc_D3.0mm_W1.6mm_P2.50mm, F.Cu at (170.7, 82.5)
- added C11: Dec_Cap, Capacitor_THT:C_Disc_D3.0mm_W1.6mm_P2.50mm, F.Cu at (66.1, 52.1)
- added C12: Dec_Cap, Capacitor_THT:C_Disc_D3.0mm_W1.6mm_P2.50mm, F.Cu at (66.1, 76.2)
- added C13: Dec_Cap, Capacitor_THT:C_Disc_D3.0mm_W1.6mm_P2.50mm, F.Cu at (68.6, 28.6)
- added C14: Dec_Cap, Capacitor_THT:C_Disc_D3.0mm_W1.6mm_P2.50mm, F.Cu at (207.0, 43.2)
- added C15: Dec_Cap, Capacitor_THT:C_Disc_D3.0mm_W1.6mm_P2.50mm, F.Cu at (203.9, 71.8)
- added C3: Dec_Cap, Capacitor_THT:C_Disc_D3.0mm_W1.6mm_P2.50mm, F.Cu at (212.1, 48.3)
- added C4: Dec_Cap, Capacitor_THT:C_Disc_D3.0mm_W1.6mm_P2.50mm, F.Cu at (129.5, 106.7)
- added C5: Dec_Cap, Capacitor_THT:C_Disc_D3.0mm_W1.6mm_P2.50mm, F.Cu at (163.8, 25.4)
- added C6: Dec_Cap, Capacitor_THT:C_Disc_D3.0mm_W1.6mm_P2.50mm, F.Cu at (181.6, 25.4)
- added C7: Dec_Cap, Capacitor_THT:C_Disc_D3.0mm_W1.6mm_P2.50mm, F.Cu at (198.1, 27.9)
- added C8: Dec_Cap, Capacitor_THT:C_Disc_D3.0mm_W1.6mm_P2.50mm, F.Cu at (163.8, 52.0)
- added C9: Dec_Cap, Capacitor_THT:C_Disc_D3.0mm_W1.6mm_P2.50mm, F.Cu at (181.6, 54.6)
- added J4: Conn_02x08_Counter_Clockwise, z80mgc:PinHeader_2x08_P2.54mm_Vertical, F.Cu at (217.2, 47.0)
- D1, D10, D11, D12, D13, D14, D15, D16, D17, D2, D3, D4, D5, D6, D7, D8, D9, DS1, R10, R11, R12, R13, R14, R15, R16, R17, R18: moved to F.Cu
- J1, J3: value Conn_02x08_Odd_Even -> Conn_02x08_Counter_Clockwise; footprint Connector_PinHeader_2.54mm:PinHeader_2x08_P2.54mm_Vertical -> z80mgc:PinHeader_2x08_P2.54mm_Vertical; moved to F.Cu
- moved R18 168.7 mm to (57.7, 158.5), turned to -90 degrees
- moved R17 165.0 mm to (61.7, 158.5), turned to -90 degrees
- moved U14 162.0 mm to (238.8, 100.3), turned to -90 degrees
- moved R16 161.5 mm to (65.8, 158.5), turned to -90 degrees
- moved C2 159.4 mm to (226.1, 104.2), turned to -90 degrees
- moved R15 158.1 mm to (69.8, 158.5), turned to -90 degrees
- moved C1 156.3 mm to (226.1, 114.3), turned to 90 degrees
- moved R14 155.1 mm to (73.9, 158.5), turned to -90 degrees
- moved R13 152.1 mm to (77.9, 158.5), turned to -90 degrees
- moved D12 149.7 mm to (94.0, 177.8), turned to -90 degrees
- moved R12 149.4 mm to (82.0, 158.5), turned to -90 degrees
- moved R11 146.9 mm to (86.0, 158.5), turned to -90 degrees
- moved D11 146.4 mm to (99.5, 177.8), turned to -90 degrees
- moved R10 144.6 mm to (90.1, 158.5), turned to -90 degrees
- moved D6 143.5 mm to (94.0, 171.9), turned to -90 degrees
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Connections:
- J1 pad 10: Net-(J1-Pin_10) -> unconnected-(J1-Pin_10-Pad10)
- J1 pad 11: Net-(J1-Pin_11) -> unconnected-(J1-Pin_11-Pad11)
- J1 pad 12: Net-(J1-Pin_12) -> unconnected-(J1-Pin_12-Pad12)
- J1 pad 13: Net-(J1-Pin_13) -> unconnected-(J1-Pin_13-Pad13)
- J1 pad 14: Net-(J1-Pin_14) -> unconnected-(J1-Pin_14-Pad14)
- J1 pad 15: Net-(J1-Pin_15) -> unconnected-(J1-Pin_15-Pad15)
- J1 pad 16: Net-(J1-Pin_16) -> unconnected-(J1-Pin_16-Pad16)
- J1 pad 9: Net-(J1-Pin_9) -> unconnected-(J1-Pin_9-Pad9)
- J3 pad 10: Net-(J3-Pin_10) -> ~{WR}
- J3 pad 11: Net-(J3-Pin_11) -> ~{CLK}
- J3 pad 12: Net-(J3-Pin_12) -> ~{CLK}
- J3 pad 13: Net-(J3-Pin_13) -> GND
- J3 pad 14: Net-(J3-Pin_14) -> GND
- J3 pad 15: Net-(J3-Pin_15) -> +5V
- J3 pad 16: Net-(J3-Pin_16) -> +5V
- J3 pad 9: Net-(J3-Pin_9) -> ~{RD}
- U1 pad 1: ADDR10 -> ADDR11
- U1 pad 16: unconnected-(U1-~{INT}-Pad16) -> +5V
- U1 pad 2: ADDR11 -> ADDR12
- U1 pad 24: unconnected-(U1-~{WAIT}-Pad24) -> +5V
- U1 pad 25: unconnected-(U1-~{BUSRQ}-Pad25) -> +5V
- U1 pad 26: unconnected-(U1-~{RESET}-Pad26) -> ~{RESET}
- U1 pad 3: ADDR12 -> ADDR13
- U1 pad 38: ADDR7 -> ADDR8
- U1 pad 39: ADDR8 -> ADDR9
- U1 pad 4: ADDR13 -> ADDR14
- U1 pad 40: ADDR9 -> ADDR10
- U1 pad 5: ADDR14 -> ADDR15
- U1 pad 6: unconnected-(U1-~{CLK}-Pad6) -> ~{CLK}
- U11 pad 11: Net-(U11-~{Y4}) -> unconnected-(U11-~{Y4}-Pad11)
- U12 pad 11: Net-(J1-Pin_8) -> Net-(J4-Pin_8)
- U12 pad 12: Net-(J1-Pin_7) -> Net-(J4-Pin_7)
- U12 pad 13: Net-(J1-Pin_6) -> Net-(J4-Pin_6)
- U12 pad 14: Net-(J1-Pin_5) -> Net-(J4-Pin_5)
- U12 pad 15: Net-(J1-Pin_4) -> Net-(J4-Pin_4)
- U12 pad 16: Net-(J1-Pin_3) -> Net-(J4-Pin_3)
- U12 pad 17: Net-(J1-Pin_2) -> Net-(J4-Pin_2)
- U12 pad 18: Net-(J1-Pin_1) -> Net-(J4-Pin_1)
- U12 pad 19: Net-(U11-~{Y1}) -> Net-(U11-~{Y2})
- U14 pad 3: unconnected-(U14-Q-Pad3) -> ~{NMI}
- U7 pad 1: ~{RD} -> GND
- U7 pad 11: Net-(J3-Pin_16) -> Net-(J1-Pin_8)
- U7 pad 12: Net-(J3-Pin_15) -> Net-(J1-Pin_7)
- U7 pad 13: Net-(J3-Pin_14) -> Net-(J1-Pin_6)
- U7 pad 14: Net-(J3-Pin_13) -> Net-(J1-Pin_5)
- U7 pad 15: Net-(J3-Pin_12) -> Net-(J1-Pin_4)
- U7 pad 16: Net-(J3-Pin_11) -> Net-(J1-Pin_3)
- U7 pad 17: Net-(J3-Pin_10) -> Net-(J1-Pin_2)
- U7 pad 18: Net-(J3-Pin_9) -> Net-(J1-Pin_1)
- U7 pad 19: Net-(U11-~{Y4}) -> Net-(U11-~{Y1})
Routing:
- net GND: track 0.00 -> 665.1 mm
- net +5V: track 0.00 -> 573.3 mm, vias 0 -> 2
- net DATA3: track 0.00 -> 323.9 mm, vias 0 -> 4
- net DATA2: track 0.00 -> 307.8 mm, vias 0 -> 4
- net DATA1: track 0.00 -> 301.9 mm, vias 0 -> 4
- net DATA0: track 0.00 -> 293.5 mm, vias 0 -> 4
- net DATA4: track 0.00 -> 278.9 mm, vias 0 -> 4
- net DATA5: track 0.00 -> 273.6 mm, vias 0 -> 4
- net ADDR14: track 0.00 -> 245.0 mm, vias 0 -> 6
- net ~{RD}: track 0.00 -> 233.0 mm, vias 0 -> 6
- net DATA6: track 48.9 -> 269.6 mm, vias 0 -> 4
- net DATA7: track 49.3 -> 269.9 mm, vias 0 -> 2
- net (no net): track 0.00 -> 199.2 mm
- net ADDR0: track 0.00 -> 171.0 mm
- net ADDR1: track 0.00 -> 170.6 mm
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- removed copper zone on B.Cu, net GND
Other:
- board outline removed
- copper layers 2 -> 4

Commit message: Work on scmenatic and PCB
Parts:
- added ?: , , F.Cu at (249.0, 131.6)
- added ?: , , F.Cu at (66.0, 18.6)
- added ?: , , F.Cu at (66.0, 131.6)
- added ?: , , F.Cu at (249.0, 18.6)
- moved D17 232.3 mm to (291.0, 52.3), turned to 0 degrees
- moved D16 231.0 mm to (291.0, 46.7), turned to 0 degrees
- moved D15 229.9 mm to (291.0, 41.2), turned to 0 degrees
- moved D14 229.1 mm to (291.0, 35.6), turned to 0 degrees
- moved D13 228.5 mm to (290.4, 29.6), turned to 0 degrees
- moved D12 225.7 mm to (285.1, 57.8), turned to 0 degrees
- moved D11 224.1 mm to (285.1, 52.3), turned to 0 degrees
- moved D10 222.7 mm to (285.1, 46.7), turned to 0 degrees
- moved D9 221.6 mm to (285.1, 41.2), turned to 0 degrees
- moved D8 220.8 mm to (285.1, 35.6), turned to 0 degrees
- moved D7 220.3 mm to (285.1, 30.1), turned to 0 degrees
- moved R18 217.9 mm to (265.8, 94.1), turned to 0 degrees
- moved D6 217.6 mm to (279.2, 57.8), turned to 0 degrees
- moved D5 215.9 mm to (279.2, 52.3), turned to 0 degrees
- moved R17 215.3 mm to (265.8, 90.1), turned to 0 degrees
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Routing:
- net GND: track 665.1 -> 1018.4 mm, vias 0 -> 8
- net (no net): track 199.2 -> 0.00 mm
- net ~{WR}: track 66.0 -> 241.7 mm
- net ADDR5: track 169.0 -> 286.2 mm, vias 0 -> 2
- net ADDR1: track 170.6 -> 283.2 mm, vias 0 -> 2
- net ADDR6: track 168.7 -> 272.2 mm, vias 0 -> 2
- net ADDR7: track 168.3 -> 271.6 mm, vias 0 -> 2
- net Net-(U4-~{CS}): track 0.00 -> 95.7 mm, vias 0 -> 2
- net ~{IORQ}: track 40.1 -> 134.6 mm, vias 0 -> 2
- net Net-(U2-~{CS}): track 3.81 -> 95.1 mm, vias 1 -> 2
- net ADDR0: track 171.0 -> 256.5 mm, vias 0 -> 2
- net ~{NMI}: track 6.35 -> 91.6 mm, vias 1 -> 2
- net Net-(DS1-E): track 0.00 -> 81.3 mm, vias 0 -> 2
- net ~{MREQ}: track 59.4 -> 122.3 mm, vias 0 -> 2
- net +5V: track 573.3 -> 636.1 mm, vias 2 -> 6
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Other:
- board outline added: 190 x 120 mm

Commit message: Work on scmenatic and PCB
Parts:
- removed ? (x4): , 
- removed the C1 at (229.9, 125.8)
- removed C10, C13, C15, C7, C8, C9: Dec_Cap, Capacitor_THT:C_Disc_D3.0mm_W1.6mm_P2.50mm
- removed J2: Conn_01x02, Connector_PinHeader_1.00mm:PinHeader_1x02_P1.00mm_Vertical
- removed the J3 at (217.2, 67.3)
- removed the U10 at (149.9, 27.9)
- removed U14: NE555P, Package_DIP:DIP-8_W7.62mm
- removed the U5 at (149.9, 54.6)
- removed the U6 at (212.1, 80.0)
- removed the U9 at (167.7, 54.6)
- added C3: 33pF, Capacitor_THT:C_Disc_D4.3mm_W1.9mm_P5.00mm, F.Cu at (124.4, 26.7)
- added C4: 0.1uf, Capacitor_THT:C_Disc_D3.0mm_W1.6mm_P2.50mm, F.Cu at (238.8, 160.0)
- added C5: 33pF, Capacitor_THT:C_Disc_D4.3mm_W1.9mm_P5.00mm, F.Cu at (124.4, 31.8)
- added CD10: 0.1uF, Capacitor_THT:C_Disc_D3.0mm_W1.6mm_P2.50mm, F.Cu at (77.3, 180.2)
- added CD11: 0.1uF, Capacitor_THT:C_Disc_D3.0mm_W1.6mm_P2.50mm, F.Cu at (77.3, 183.3)
- added CD12: 0.1uF, Capacitor_THT:C_Disc_D3.0mm_W1.6mm_P2.50mm, F.Cu at (77.3, 189.6)
- added CD6: 0.1uF, Capacitor_THT:C_Disc_D3.0mm_W1.6mm_P2.50mm, F.Cu at (158.8, 235.0)
- added CD9: 0.1uF, Capacitor_THT:C_Disc_D3.0mm_W1.6mm_P2.50mm, F.Cu at (77.3, 186.5)
- added J4: POWER, Connector_PinHeader_1.00mm:PinHeader_1x02_P1.00mm_Vertical, F.Cu at (52.3, 204.1)
- added J5: RESET, Connector_PinHeader_1.00mm:PinHeader_1x02_P1.00mm_Vertical, F.Cu at (55.7, 204.1)
- added J6: IO_EXP, z80mgc:PinHeader_2x08_P2.54mm_Vertical, F.Cu at (121.9, 258.1)
- added R21: 10k, Resistor_THT:R_Axial_DIN0207_L6.3mm_D2.5mm_P10.16mm_Horizontal, F.Cu at (243.8, 157.5)
- added R22: 1k, Resistor_THT:R_Axial_DIN0207_L6.3mm_D2.5mm_P10.16mm_Horizontal, F.Cu at (229.9, 143.5)
- added R23: 1k, Resistor_THT:R_Axial_DIN0207_L6.3mm_D2.5mm_P10.16mm_Horizontal, F.Cu at (67.3, 212.1)
- added RN1: R_Network08, Resistor_THT:R_Array_SIP9, F.Cu at (240.0, 82.6)
- added RN2: R_Network08, Resistor_THT:R_Array_SIP9, F.Cu at (236.2, 12.7)
- added U12: NE555P, Package_DIP:DIP-8_W7.62mm, F.Cu at (231.2, 148.6)
- added U2: 74HC00, Package_DIP:DIP-14_W7.62mm_Socket_LongPads, F.Cu at (167.7, 52.1)
- added U3: 74HC04, Package_DIP:DIP-14_W7.62mm_Socket_LongPads, F.Cu at (148.6, 27.9)
- added U4: 74HC02, Package_DIP:DIP-14_W7.62mm_Socket_LongPads, F.Cu at (167.6, 27.9)
- C1: renamed from C5; value Dec_Cap -> 0.1uF
- C2: value C_Polarized -> 1uF
- CD1: renamed from C6; value Dec_Cap -> 0.1uF
- CD2: renamed from C3; value Dec_Cap -> 0.1uF
- CD3: renamed from C4; value Dec_Cap -> 0.1uF
- CD4: renamed from C12; value Dec_Cap -> F
- CD5: renamed from C11; value Dec_Cap -> 0.1uF
- CD7: renamed from C14; value Dec_Cap -> 0.1uF
- J1: renamed from J4; value Conn_02x08_Counter_Clockwise -> IO_A
- J3: renamed from J1; value Conn_02x08_Counter_Clockwise -> IO_BTN
- R19: value 10k -> 100k
- R20: value 1k -> 260; footprint Resistor_THT:R_Axial_DIN0207_L6.3mm_D2.5mm_P10.16mm_Horizontal -> Resistor_THT:R_Axial_DIN0204_L3.6mm_D1.6mm_P5.08mm_Horizontal
- U8: value 74HC02 -> 74HC86
- Y1: value Crystal -> 6MHz
- moved R20 134.8 mm to (134.6, 31.8)
- moved R19 114.5 mm to (138.4, 34.3), turned to 90 degrees
- moved U8 31.8 mm to (186.7, 53.3)
- moved C2 25.7 mm to (226.1, 151.1), turned to 90 degrees
- moved CD1 3.82 mm to (182.9, 25.4)
- moved Y1 3.73 mm to (129.5, 26.7)
- moved C1 2.55 mm to (163.8, 25.4)
- renumbered U1 to CPU1, D9 to D10, D10 to D11, D11 to D12, D12 to D13, D13 to D14, D14 to D9, R2 to R10, R3 to R11, R4 to R12, R5 to R13, R6 to R14, R7 to R15, R8 to R16, R9 to R17, R15 to R18, R10 to R2, R11 to R3, R12 to R4, R13 to R5, R14 to R6, R16 to R7, R17 to R8, R18 to R9, U4 to U1, U12 to U10, U2 to U5, U3 to U6, U11 to U7, U7 to U9
Connections:
- J1 pad 10: unconnected-(J4-Pin_10-Pad10) -> GND
- J1 pad 11: unconnected-(J4-Pin_11-Pad11) -> GND
- J1 pad 12: unconnected-(J4-Pin_12-Pad12) -> GND
- J1 pad 13: unconnected-(J4-Pin_13-Pad13) -> GND
- J1 pad 14: unconnected-(J4-Pin_14-Pad14) -> GND
- J1 pad 15: unconnected-(J4-Pin_15-Pad15) -> GND
- J1 pad 16: unconnected-(J4-Pin_16-Pad16) -> GND
- J1 pad 9: unconnected-(J4-Pin_9-Pad9) -> GND
- J3 pad 10: unconnected-(J1-Pin_10-Pad10) -> GND
- J3 pad 11: unconnected-(J1-Pin_11-Pad11) -> GND
- J3 pad 12: unconnected-(J1-Pin_12-Pad12) -> GND
- J3 pad 13: unconnected-(J1-Pin_13-Pad13) -> GND
- J3 pad 14: unconnected-(J1-Pin_14-Pad14) -> GND
- J3 pad 15: unconnected-(J1-Pin_15-Pad15) -> GND
- J3 pad 16: unconnected-(J1-Pin_16-Pad16) -> GND
- J3 pad 9: unconnected-(J1-Pin_9-Pad9) -> GND
- R19 pad 2: +5V -> Net-(C3-Pad1)
- R20 pad 1: Net-(U14-THR) -> Net-(C5-Pad1)
- U10 pad 1: GND -> ~{RD}
- U7 pad 11: unconnected-(U11-~{Y4}-Pad11) -> Net-(J6-Pin_15)
- U7 pad 15: Net-(U11-~{Y0}) -> Net-(U7-~{Y0})
- U8 pad 1: Net-(U10-Pad10) -> ADDR1
- U8 pad 10: unconnected-(U8-Pad10) -> GND
- U8 pad 11: Net-(U5-Pad11) -> unconnected-(U8-Pad11)
- U8 pad 12: Net-(U11-~{Y0}) -> GND
- U8 pad 13: Net-(DS1-E) -> GND
- U8 pad 2: ~{MREQ} -> ~{WR}
- U8 pad 3: ADDR15 -> Net-(U4-Pad8)
- U8 pad 4: Net-(U10-Pad12) -> GND
- U8 pad 5: ADDR14 -> GND
- U8 pad 6: Net-(U10-Pad8) -> unconnected-(U8-Pad6)
- U8 pad 8: GND -> unconnected-(U8-Pad8)
- Y1 pad 1: unconnected-(Y1-Pad1) -> Net-(C3-Pad1)
- Y1 pad 2: unconnected-(Y1-Pad2) -> Net-(C5-Pad1)
Routing:
- net +5V: track 636.1 -> 402.0 mm, vias 6 -> 1
- net GND: track 1018.4 -> 863.0 mm, vias 8 -> 4
- net ADDR5: track 286.2 -> 172.8 mm, vias 2 -> 0
- net ADDR15: track 130.6 -> 23.3 mm, vias 4 -> 1
- net ADDR7: track 271.6 -> 172.2 mm, vias 2 -> 0
- net ADDR14: track 256.9 -> 161.4 mm, vias 6 -> 3
- net ~{IORQ}: track 134.6 -> 40.6 mm, vias 2 -> 0
- net Net-(U5-~{CS}): track 95.1 -> 5.61 mm, vias 2 -> 1
- net ADDR6: track 272.2 -> 186.9 mm, vias 2 -> 1
- net ~{MREQ}: track 122.3 -> 40.6 mm, vias 2 -> 0
- net Net-(DS1-E): track 81.3 -> 4.56 mm, vias 2 -> 0
- net ~{WR}: track 241.7 -> 182.1 mm
- net Net-(U1-~{CS}): track 95.7 -> 42.6 mm, vias 2 -> 1
- net Net-(U5-Pad11): track 51.2 -> 0.00 mm, vias 2 -> 0
- net ~{RD}: track 291.8 -> 258.9 mm
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
Commit message: Snake working with framebuffer
Parts:
- removed R10, R11, R12, R13, R14, R15, R16, R17, R6, R7, R8, R9: 1k, Resistor_THT:R_Axial_DIN0207_L6.3mm_D2.5mm_P10.16mm_Horizontal
- added ?: , , F.Cu at (65.5, 132.1)
- added ?: , clipboard:a9ab44e1-df2f-4d8c-8125-f91eaead8355, F.Cu at (65.5, 17.8)
- added ?: , , F.Cu at (249.5, 18.1)
- added ?: , , F.Cu at (249.5, 132.1)
- added RN3: 1k, Resistor_THT:R_Array_SIP9, F.Cu at (276.9, 91.4)
- added RN4: 1k, Resistor_THT:R_Array_SIP9, F.Cu at (264.2, 114.3)
- J4: footprint Connector_PinHeader_1.00mm:PinHeader_1x02_P1.00mm_Vertical -> Connector_PinHeader_2.54mm:PinHeader_1x02_P2.54mm_Vertical
- J5: footprint Connector_PinHeader_1.00mm:PinHeader_1x02_P1.00mm_Vertical -> Connector_PinSocket_2.54mm:PinSocket_1x02_P2.54mm_Vertical
- RN1, RN2: value R_Network08 -> 10k
- U5, U6: footprint Package_DIP:DIP-28_W15.24mm_Socket_LongPads -> Package_DIP:DIP-28_W15.24mm_LongPads
- moved J6 200.8 mm to (214.6, 80.0), turned to 90 degrees
- moved CD9 200.1 mm to (199.4, 27.9), turned to 90 degrees
- moved D11 185.3 mm to (119.4, 129.5), turned to 90 degrees
- moved D10 182.3 mm to (125.7, 129.5), turned to 90 degrees
- moved CD10 176.1 mm to (198.1, 52.0), turned to 90 degrees
- moved J4 175.4 mm to (198.1, 106.7)
- moved D12 167.3 mm to (128.3, 110.5), turned to 180 degrees
- moved R2 164.5 mm to (114.3, 125.7), turned to 180 degrees
- moved R3 164.4 mm to (114.3, 129.5), turned to 180 degrees
- moved D13 163.6 mm to (128.3, 104.1), turned to 180 degrees
- moved CD11 153.4 mm to (179.1, 68.6)
- moved R4 146.1 mm to (123.2, 101.6), turned to 180 degrees
- moved R5 144.6 mm to (123.2, 97.8), turned to 180 degrees
- moved CD12 144.1 mm to (180.3, 88.9), turned to 90 degrees
- moved CD6 140.5 mm to (221.4, 109.2)
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- renumbered C1 to CD13
Connections:
- DS1 pad 6: Net-(DS1-E) -> DISP_EN
- RN1 pad 2: Net-(J3-Pin_8) -> Net-(J3-Pin_1)
- RN1 pad 3: Net-(J3-Pin_7) -> Net-(J3-Pin_2)
- RN1 pad 4: Net-(J3-Pin_6) -> Net-(J3-Pin_3)
- RN1 pad 5: Net-(J3-Pin_5) -> Net-(J3-Pin_4)
- RN1 pad 6: Net-(J3-Pin_4) -> Net-(J3-Pin_5)
- RN1 pad 7: Net-(J3-Pin_3) -> Net-(J3-Pin_6)
- RN1 pad 8: Net-(J3-Pin_2) -> Net-(J3-Pin_7)
- RN1 pad 9: Net-(J3-Pin_1) -> Net-(J3-Pin_8)
- RN2 pad 2: Net-(J1-Pin_8) -> Net-(J1-Pin_1)
- RN2 pad 3: Net-(J1-Pin_7) -> Net-(J1-Pin_2)
- RN2 pad 4: Net-(J1-Pin_6) -> Net-(J1-Pin_3)
- RN2 pad 5: Net-(J1-Pin_5) -> Net-(J1-Pin_4)
- RN2 pad 6: Net-(J1-Pin_4) -> Net-(J1-Pin_5)
- RN2 pad 7: Net-(J1-Pin_3) -> Net-(J1-Pin_6)
- RN2 pad 8: Net-(J1-Pin_2) -> Net-(J1-Pin_7)
- RN2 pad 9: Net-(J1-Pin_1) -> Net-(J1-Pin_8)
- U1 pad 20: Net-(U1-~{CS}) -> ~{RAM1_EN}
- U2 pad 1: ADDR15 -> Net-(U2-Pad1)
- U2 pad 10: ~{WR} -> +5V
- U2 pad 11: unconnected-(U2-Pad11) -> Net-(U7-E3)
- U2 pad 12: GND -> ~{RD}
- U2 pad 13: GND -> ~{WR}
- U2 pad 2: Net-(U2-Pad2) -> ADDR15
- U2 pad 3: Net-(U1-~{CS}) -> ~{RAM1_EN}
- U2 pad 6: Net-(U6-~{CS}) -> ~{ROM2_EN}
- U2 pad 8: Net-(U7-E3) -> unconnected-(U2-Pad8)
- U2 pad 9: ~{RD} -> +5V
- U3 pad 1: Net-(C3-Pad1) -> ~{ROM1_EN}
- U3 pad 10: Net-(U5-~{CS}) -> Net-(U2-Pad1)
- U3 pad 11: Net-(U3-Pad11) -> ~{MREQ}
- U3 pad 12: unconnected-(U3-Pad12) -> Net-(U3-Pad12)
- U3 pad 13: GND -> Net-(U2-Pad4)
- U3 pad 2: Net-(R19-Pad1) -> Net-(U5-~{CS})
- U3 pad 3: Net-(R19-Pad1) -> Net-(C3-Pad1)
- U3 pad 4: ~{CLK} -> Net-(R19-Pad1)
- U3 pad 5: ~{MREQ} -> Net-(R19-Pad1)
- U3 pad 6: Net-(U2-Pad2) -> ~{CLK}
- U3 pad 8: Net-(U3-Pad8) -> unconnected-(U3-Pad8)
- U3 pad 9: Net-(U2-Pad4) -> GND
- U4 pad 1: Net-(U2-Pad4) -> ~{ROM1_EN}
- U4 pad 10: Net-(DS1-E) -> unconnected-(U4-Pad10)
- U4 pad 11: GND -> Net-(U4-Pad11)
- U4 pad 12: GND -> Net-(U7-~{Y0})
- U4 pad 13: unconnected-(U4-Pad13) -> DISP_EN
- U4 pad 2: ~{MREQ} -> ADDR14
- U4 pad 3: ADDR15 -> Net-(U3-Pad12)
- U4 pad 4: Net-(U3-Pad11) -> Net-(U2-Pad4)
- U4 pad 5: ADDR14 -> ~{MREQ}
- U4 pad 6: Net-(U3-Pad8) -> ADDR15
- U4 pad 8: Net-(U4-Pad8) -> +5V
- U4 pad 9: Net-(U7-~{Y0}) -> +5V
- U5 pad 1: ADDR14 -> unconnected-(U5-~{BSY}-Pad1)
- U5 pad 26: ADDR13 -> unconnected-(U5-NC-Pad26)
- U6 pad 1: ADDR14 -> unconnected-(U6-~{BSY}-Pad1)
- U6 pad 14: GND -> unconnected-(U6-GND-Pad14)
- U6 pad 20: Net-(U6-~{CS}) -> ~{ROM2_EN}
- U6 pad 26: ADDR13 -> unconnected-(U6-NC-Pad26)
- U8 pad 10: GND -> +5V
- U8 pad 12: GND -> +5V
- U8 pad 13: GND -> +5V
- U8 pad 3: Net-(U4-Pad8) -> Net-(U4-Pad11)
- U8 pad 4: GND -> +5V
- U8 pad 5: GND -> +5V
- U8 pad 9: GND -> +5V
Routing:
- net +5V: track 402.0 -> 561.0 mm, vias 1 -> 0
- net ~{WR}: track 182.1 -> 39.2 mm, vias 4 -> 3
- net GND: track 863.0 -> 993.5 mm, vias 4 -> 0
- net ~{RD}: track 258.9 -> 141.3 mm, vias 6 -> 5
- net Net-(U6-~{CS}): track 72.6 -> 0.00 mm, vias 1 -> 0
- net ~{RESET}: track 0.00 -> 62.8 mm
- net DISP_EN: track 0.00 -> 62.3 mm
- net ~{NMI}: track 62.9 -> 3.81 mm
- net Net-(U2-Pad4): track 0.00 -> 50.1 mm
- net ADDR14: track 161.4 -> 204.8 mm
- net ADDR1: track 263.6 -> 220.5 mm
- net Net-(U1-~{CS}): track 42.6 -> 0.00 mm, vias 1 -> 0
- net Net-(J6-Pin_16): track 41.1 -> 0.00 mm, vias 1 -> 0
- net Net-(U7-E3): track 0.00 -> 39.0 mm
- net Net-(U4-Pad11): track 0.00 -> 33.2 mm
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Other:
- board text added: "Martin Bernardi"
- board text added: "v1.0"
- board text added: "z80mgc"

Commit message: Lots of work on Kicad, and gave up on PCB
Parts:
- added J10: ~{WAIT}, Connector_PinHeader_1.27mm:PinHeader_1x01_P1.27mm_Vertical, F.Cu at (259.1, 114.9)
- added J11: ~{CLK}, Connector_PinHeader_1.27mm:PinHeader_1x01_P1.27mm_Vertical, F.Cu at (172.1, 106.7)
- added J12: ~{RFSH}, TestPoint:TestPoint_THTPad_D2.0mm_Drill1.0mm, F.Cu at (151.1, 129.5)
- added J13: ~{RFSH}, Connector_PinHeader_1.27mm:PinHeader_1x01_P1.27mm_Vertical, F.Cu at (317.7, 68.7)
- added J14: ~{BUSRQ}, Connector_PinHeader_1.27mm:PinHeader_1x01_P1.27mm_Vertical, F.Cu at (317.7, 72.0)
- added J15: ~{RESET}, Connector_PinHeader_1.27mm:PinHeader_1x01_P1.27mm_Vertical, F.Cu at (317.7, 75.4)
- added J16: ~{RD}, Connector_PinHeader_1.27mm:PinHeader_1x01_P1.27mm_Vertical, F.Cu at (317.7, 78.7)
- added J17: ~{WR}, Connector_PinHeader_1.27mm:PinHeader_1x01_P1.27mm_Vertical, F.Cu at (321.9, 65.3)
- added J18: ~{MREQ}, Connector_PinHeader_1.27mm:PinHeader_1x01_P1.27mm_Vertical, F.Cu at (321.9, 68.7)
- added J19: ~{IORQ}, Connector_PinHeader_1.27mm:PinHeader_1x01_P1.27mm_Vertical, F.Cu at (321.9, 72.0)
- added J2: USB_B, Connector_USB:USB_B_OST_USB-B1HSxx_Horizontal, F.Cu at (306.6, 113.1)
- added J20: ~{BUSACK}, Connector_PinHeader_1.27mm:PinHeader_1x01_P1.27mm_Vertical, F.Cu at (321.9, 75.4)
- added J7: ~{M1}, Connector_PinHeader_1.27mm:PinHeader_1x01_P1.27mm_Vertical, F.Cu at (168.9, 139.7)
- added J8: ~{NMI}, Connector_PinHeader_1.27mm:PinHeader_1x01_P1.27mm_Vertical, F.Cu at (313.6, 68.7)
- added J9: ~{HALT}, TestPoint:TestPoint_THTPad_D2.0mm_Drill1.0mm, F.Cu at (325.8, 78.7)
- added R2: 10k, Resistor_THT:R_Axial_DIN0207_L6.3mm_D2.5mm_P10.16mm_Horizontal, F.Cu at (325.5, 65.7)
- added R3: 10k, Resistor_THT:R_Axial_DIN0207_L6.3mm_D2.5mm_P10.16mm_Horizontal, F.Cu at (249.6, 109.2)
- added R4: 10k, Resistor_THT:R_Axial_DIN0207_L6.3mm_D2.5mm_P10.16mm_Horizontal, F.Cu at (325.5, 73.8)
- added RN5: 1k, Resistor_THT:R_Array_SIP7, F.Cu at (214.6, 16.5)
- added RN6: 1k, Resistor_THT:R_Array_SIP7, F.Cu at (214.6, 48.3)
- moved D15 94.0 mm to (243.8, 83.2)
- moved D16 89.2 mm to (243.8, 78.1)
- moved D14 85.9 mm to (243.8, 88.3)
- moved D17 85.3 mm to (243.8, 73.0)
- moved D6 75.5 mm to (246.4, 55.9), turned to 180 degrees
- moved D7 75.4 mm to (246.4, 61.0), turned to 180 degrees
- moved D3 67.1 mm to (246.4, 40.6), turned to 180 degrees
- moved D4 67.1 mm to (246.4, 45.7), turned to 180 degrees
- moved D5 67.0 mm to (246.4, 50.8), turned to 180 degrees
- moved D2 62.1 mm to (246.4, 35.6), turned to 180 degrees
- moved D1 62.0 mm to (246.4, 30.5), turned to 180 degrees
- moved RN4 61.3 mm to (250.2, 54.6), turned to 90 degrees
- moved D0 55.2 mm to (246.4, 25.4), turned to 180 degrees
- moved RN3 28.5 mm to (250.2, 101.6), turned to 90 degrees
- moved U10 8.90 mm to (212.1, 72.4)
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- renumbered D1 to D0, D2 to D1, D3 to D2, D4 to D3, D5 to D4, D6 to D5, D7 to D6, D8 to D7
Connections:
- CPU1 pad 16: +5V -> ~{INT}
- CPU1 pad 18: unconnected-(CPU1-~{HALT}-Pad18) -> ~{HALT}
- CPU1 pad 23: unconnected-(CPU1-~{BUSACK}-Pad23) -> ~{BUSACK}
- CPU1 pad 24: +5V -> ~{WAIT}
- CPU1 pad 25: +5V -> ~{BUSRQ}
- CPU1 pad 27: unconnected-(CPU1-~{M1}-Pad27) -> ~{M1}
- CPU1 pad 28: unconnected-(CPU1-~{RFSH}-Pad28) -> ~{RFSH}
- J1 pad 11: GND -> Net-(J1-Pin_11)
- J1 pad 12: GND -> Net-(J1-Pin_12)
- J1 pad 13: GND -> Net-(J1-Pin_13)
- J1 pad 14: GND -> Net-(J1-Pin_14)
- J1 pad 15: GND -> Net-(J1-Pin_15)
- J1 pad 16: GND -> Net-(J1-Pin_16)
- J3 pad 11: GND -> Net-(J3-Pin_11)
- J3 pad 12: GND -> Net-(J3-Pin_12)
- J3 pad 13: GND -> Net-(J3-Pin_13)
- J3 pad 14: GND -> Net-(J3-Pin_14)
- J3 pad 15: GND -> Net-(J3-Pin_15)
- J3 pad 16: GND -> Net-(J3-Pin_16)
Routing:
- net GND: track 993.5 -> 924.6 mm
- net +5V: track 561.0 -> 582.9 mm
- net Net-(D7-K): track 0.00 -> 10.5 mm
- net Net-(D0-K): track 0.00 -> 10.5 mm
- net Net-(U10-CE): track 8.15 -> 0.00 mm
- net Net-(D6-K): track 0.00 -> 7.93 mm
- net Net-(D1-K): track 0.00 -> 7.93 mm
- net Net-(D5-K): track 0.00 -> 6.13 mm
- net Net-(D2-K): track 0.00 -> 6.13 mm
- net Net-(J1-Pin_16): track 0.00 -> 5.08 mm
- net Net-(J1-Pin_15): track 0.00 -> 5.08 mm
- net Net-(J1-Pin_14): track 0.00 -> 5.08 mm
- net Net-(J1-Pin_13): track 0.00 -> 5.08 mm
- net Net-(J1-Pin_12): track 0.00 -> 5.08 mm
- net Net-(J1-Pin_11): track 0.00 -> 5.08 mm
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